File: FXDSP.kicad_pcb (KiCad board)
At the start: 4 copper layers, 54.6 x 96.5 mm, 125 parts, among them J101 Barrel_Jack_Switch, J201 Conn_01x10, J202 Conn_01x07, J203 Conn_ARM_JTAG_SWD_10, J204 USB_C_Receptacle_USB2.0, J301 AudioJack3_Switch, J302 AudioJack3_Switch, K301 G6K-2, K302 G6K-2, Q101 Si2301CDS, Q301 MMBT3904, Q302 MMBT3904, SW201 SW_Push, U101 NCP1117-5.0, U102 NCP1117-3.3, U201 STM32F405RGTx, U301 PCM3060, U302 NE5532, U303 NE5532, U304 NE5532, Y201 12.288Mhz

Commit message: Fix reset problems from r01 PCB
Parts:
- removed R204: 1k, Resistor_SMD:R_0402_1005Metric
- added C211: 100n, Capacitor_SMD:C_0402_1005Metric, F.Cu at (125.1, 63.5)
- moved C208 0.51 mm to (135.4, 70.1)
- moved G*** 0.25 mm to (127.0, 121.7)
Connections:
- U301 pad 15: GND -> +3.3V
Routing:
- net +3.3V: track 29.7 -> 37.4 mm, vias 10 -> 12
- net GND: track 68.6 -> 66.7 mm, vias 131 -> 130
- net +5VA: track 4.19 -> 5.33 mm, vias 8 -> 9
- net /Audio/BYPASSL: track 66.7 -> 65.7 mm
- net /Audio/BYPASSR: track 100.6 -> 99.7 mm
