File: audio.kicad_sch (KiCad schematic)
At the start: 69 parts, among them J1 AudioJack3_Switch, J2 AudioJack3_Switch, K301 G6K-2, K302 G6K-2, Q301 MMBT3904, Q302 MMBT3904, U2 NE5532, U3 NE5532, U4 PCM3060, U5 NE5532

Commit message: Fix reset problems from r01 PCB
Connections:
- net +3.3V: now also U4.15 (~{RST})
- net GND: no longer U4.15 (~{RST})
Changed lines of the file:
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@@
   (title_block
     (title "Whatever DSP")
+    (date "2023-05-14")
     (rev "${REVISION}")
     (company "Nuclear Lighthouse Studios")
@@
     (stroke (width 0) (type solid))
   )
-  (wire (pts (xy 53.34 88.265) (xy 53.34 86.995))
-    (stroke (width 0) (type default))
-  )
   (wire (pts (xy 28.575 113.665) (xy 29.845 113.665))
     (stroke (width 0) (type default))
@@
   (wire (pts (xy 33.655 168.91) (xy 34.925 168.91))
     (stroke (width 0) (type solid))
+  )
+  (wire (pts (xy 53.34 85.725) (xy 53.34 86.995))
+    (stroke (width 0) (type default))
   )
   (wire (pts (xy 63.5 175.26) (xy 73.66 175.26))
@@
         (path "/e63e39d7-6ac0-4ffd-8aa3-1841a4541b55/f63d5912-408b-480e-94bc-e00855e13fae"
           (reference "#PWR0304") (unit 1)
-        )
-      )
-    )
-  )
-  (symbol (lib_id "power:GND") (at 53.34 88.265 0) (unit 1)
-    (in_bom yes) (on_board yes) (dnp no) (fields_autoplaced)
-    (property "Reference" "#PWR0313" (at 53.34 94.615 0)
-      (effects (font (size 1.27 1.27)) hide)
-    )
-    (property "Value" "GND" (at 53.34 93.345 0)
-      (effects (font (size 1.27 1.27)))
-    )
-    (property "Footprint" "" (at 53.34 88.265 0)
-      (effects (font (size 1.27 1.27)) hide)
-    )
-    (property "Datasheet" "" (at 53.34 88.265 0)
-      (effects (font (size 1.27 1.27)) hide)
-    )
-    (pin "1")
-    (instances
-      (project "FXDSP"
-        (path "/e63e39d7-6ac0-4ffd-8aa3-1841a4541b55/f63d5912-408b-480e-94bc-e00855e13fae"
-          (reference "#PWR0313") (unit 1)
         )
       )
@@
         )
       )
+    )
+  )
+  (symbol (lib_id "power:+3.3V") (at 53.34 85.725 0) (unit 1)
+    (in_bom yes) (on_board yes) (dnp no) (fields_autoplaced)
+    (property "Reference" "#PWR0339" (at 53.34 89.535 0)
+      (effects (font (size 1.27 1.27)) hide)
+    )
+    (property "Value" "+3.3V" (at 53.34 81.915 0)
+      (effects (font (size 1.27 1.27)))
+    )
+    (property "Footprint" "" (at 53.34 85.725 0)
+      (effects (font (size 1.27 1.27)) hide)
+    )
+    (property "Datasheet" "" (at 53.34 85.725 0)
+      (effects (font (size 1.27 1.27)) hide)
+    )
+    (pin "1")
+    (instances
+      (project "FXDSP"
+        (path "/e63e39d7-6ac0-4ffd-8aa3-1841a4541b55/f63d5912-408b-480e-94bc-e00855e13fae"
+          (reference "#PWR0339") (unit 1)
+        )
+      )
