File: digital.kicad_sch (KiCad schematic)
At the start: 27 parts, among them J3 Conn_ARM_JTAG_SWD_10, J4 USB_C_Receptacle_USB2.0, J5 Conn_01x10, J6 Conn_01x07, SW1 SW_Push, U1 STM32F405RGTx, Y1 12.288Mhz

Commit message: Fix reset problems from r01 PCB
Parts:
- removed R4: 1k, Resistor_SMD:R_0402_1005Metric, symbol Device:R
- added C35: 100n, Capacitor_SMD:C_0402_1005Metric, symbol Device:C
Connections:
- net GND: now also C35.2
- net NRST: now also C35.1
Other:
- company: (none) -> Nuclear Lighthouse Studios
- title: (none) -> Whatever DSP
Changed lines of the file:
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@@
 (kicad_sch (version 20230121) (generator eeschema)
   (paper "A4")
+  (title_block
+    (title "Whatever DSP")
+    (date "2023-05-14")
+    (rev "${REVISION}")
+    (company "Nuclear Lighthouse Studios")
+    (comment 1 "${LICENSE}")
+  )
   (junction (at 133.35 48.26) (diameter 0) (color 0 0 0 0)
   )
@@
         (path "/e63e39d7-6ac0-4ffd-8aa3-1841a4541b55/54e2d0aa-21e2-4e7a-91a5-58f6e6fcfb6d"
           (reference "C204") (unit 1)
+        )
+      )
+    )
+  )
+  (symbol (lib_id "Device:C") (at 128.27 48.26 270) (unit 1)
+    (in_bom yes) (on_board yes) (dnp no) (fields_autoplaced)
+    (property "Reference" "C35" (at 128.27 41.91 90)
+      (effects (font (size 1.27 1.27)))
+    )
+    (property "Value" "100n" (at 128.27 44.45 90)
+      (effects (font (size 1.27 1.27)))
+    )
+    (property "Footprint" "Capacitor_SMD:C_0402_1005Metric" (at 124.46 49.2252 0)
+      (effects (font (size 1.27 1.27)) hide)
+    )
+    (property "Datasheet" "~" (at 128.27 48.26 0)
+      (effects (font (size 1.27 1.27)) hide)
+    )
+    (pin "1")
+    (pin "2")
+    (instances
+      (project "FXDSP"
+        (path "/e63e39d7-6ac0-4ffd-8aa3-1841a4541b55"
+          (reference "C35") (unit 1)
+        )
+        (path "/e63e39d7-6ac0-4ffd-8aa3-1841a4541b55/54e2d0aa-21e2-4e7a-91a5-58f6e6fcfb6d"
+          (reference "C211") (unit 1)
         )
       )
@@
         )
       )
-    )
-  )
-  (symbol (lib_id "Device:R") (at 128.27 48.26 270) (unit 1)
-    (in_bom yes) (on_board yes) (dnp no)
-    (property "Reference" "R4" (at 128.27 43.0022 90)
-      (effects (font (size 1.27 1.27)))
-    )
-    (property "Value" "1k" (at 128.27 45.3136 90)
-      (effects (font (size 1.27 1.27)))
-    )
-    (property "Footprint" "Resistor_SMD:R_0402_1005Metric" (at 128.27 46.482 90)
-      (effects (font (size 1.27 1.27)) hide)
-    )
-    (property "Datasheet" "~" (at 128.27 48.26 0)
-      (effects (font (size 1.27 1.27)) hide)
-    )
-    (pin "1")
-    (pin "2")
-    (instances
-      (project "FXDSP"
-        (path "/e63e39d7-6ac0-4ffd-8aa3-1841a4541b55"
-          (reference "R4") (unit 1)
-        )
-        (path "/e63e39d7-6ac0-4ffd-8aa3-1841a4541b55/54e2d0aa-21e2-4e7a-91a5-58f6e6fcfb6d"
-          (reference "R204") (unit 1)
-        )
-      )
