File: Interface PCBs/PotBoard/PotBoard.kicad_pcb (KiCad board)
At the start: 2 copper layers, 54.6 x 52.7 mm, 11 parts, among them J101 Conn_01x10, J102 Conn_01x07

Commit message: Correct positioning of lower potentiometers on interface PCB
Parts:
- moved RV104 2.54 mm to (104.7, 89.5)
- moved RV105 2.54 mm to (131.4, 89.5)
Routing:
- net +3.3VA: track 104.9 -> 107.0 mm
- net ADC_IN_4: track 39.4 -> 37.6 mm
Changed lines of the file:
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@@
   )
   (footprint "Potentiometer_THT:Potentiometer_Alps_RK09K_Single_Vertical" (layer "F.Cu")
-    (at 104.735 86.995 -90)
+    (at 104.735 89.535 -90)
     (descr "113004U 1130A6S 11300DR 1130A8G 1130081 1130A5R 1130AP5 1130AST  D1130C3W D1130C1B D1130C3C D1130C2P Potentiometer, vertical, Alps RK09K Single, https://tech.alpsalpine.com/prod/e/pdf/potentiometer/rotarypotentiometers/rk09k/rk09k.pdf")
     (tags "Potentiometer vertical Alps RK09K RK09D Single Snapin")
@@
   )
   (footprint "Potentiometer_THT:Potentiometer_Alps_RK09K_Single_Vertical" (layer "F.Cu")
-    (at 131.405 86.995 -90)
+    (at 131.405 89.535 -90)
     (descr "113004U 1130A6S 11300DR 1130A8G 1130081 1130A5R 1130AP5 1130AST  D1130C3W D1130C1B D1130C3C D1130C2P Potentiometer, vertical, Alps RK09K Single, https://tech.alpsalpine.com/prod/e/pdf/potentiometer/rotarypotentiometers/rk09k/rk09k.pdf")
     (tags "Potentiometer vertical Alps RK09K RK09D Single Snapin")
@@
   (gr_line (start 138.43 53.34) (end 120.015 53.34)
     (stroke (width 0.15) (type default)) (layer "Edge.Cuts"))
-  (segment (start 124.5 85.09) (end 126.405 86.995) (width 0.5) (layer "F.Cu") (net 11))
-  (segment (start 99.735 86.995) (end 101.64 85.09) (width 0.5) (layer "F.Cu") (net 11))
+  (segment (start 99.735 87.67) (end 99.735 89.535) (width 0.5) (layer "F.Cu") (net 11))
+  (segment (start 93.345 81.28) (end 99.735 87.67) (width 0.5) (layer "F.Cu") (net 11))
+  (segment (start 101.64 87.63) (end 124.5 87.63) (width 0.5) (layer "F.Cu") (net 11))
   (segment (start 104.18 81.28) (end 113.07 72.39) (width 0.5) (layer "F.Cu") (net 11))
   (segment (start 95.27 64.79) (end 99.735 60.325) (width 0.5) (layer "F.Cu") (net 11))
   (segment (start 93.345 81.28) (end 95.27 79.355) (width 0.5) (layer "F.Cu") (net 11))
-  (segment (start 93.345 81.28) (end 94.02 81.28) (width 0.5) (layer "F.Cu") (net 11))
+  (segment (start 124.5 87.63) (end 126.405 89.535) (width 0.5) (layer "F.Cu") (net 11))
   (segment (start 113.07 72.39) (end 125.135 60.325) (width 0.5) (layer "F.Cu") (net 11))
   (segment (start 95.27 79.355) (end 95.27 64.79) (width 0.5) (layer "F.Cu") (net 11))
   (segment (start 125.135 60.325) (end 126.405 60.325) (width 0.5) (layer "F.Cu") (net 11))
   (segment (start 92.075 81.28) (end 104.18 81.28) (width 0.5) (layer "F.Cu") (net 11))
-  (segment (start 101.64 85.09) (end 124.5 85.09) (width 0.5) (layer "F.Cu") (net 11))
-  (segment (start 94.02 81.28) (end 99.735 86.995) (width 0.5) (layer "F.Cu") (net 11))
+  (segment (start 99.735 89.535) (end 101.64 87.63) (width 0.5) (layer "F.Cu") (net 11))
   (segment (start 92.075 81.28) (end 93.345 81.28) (width 0.5) (layer "F.Cu") (net 11))
   (segment (start 114.935 70.485) (end 115.57 71.12) (width 0.5) (layer "B.Cu") (net 12))
@@
   (segment (start 121.92 75.565) (end 128.905 68.58) (width 0.5) (layer "B.Cu") (net 13))
   (segment (start 92.075 86.36) (end 95.885 86.36) (width 0.5) (layer "B.Cu") (net 13))
-  (segment (start 92.075 88.9) (end 101.602792 88.9) (width 0.5) (layer "B.Cu") (net 14))
-  (segment (start 101.602792 88.9) (end 102.235 88.267792) (width 0.5) (layer "B.Cu") (net 14))
-  (segment (start 102.235 88.267792) (end 102.235 86.995) (width 0.5) (layer "B.Cu") (net 14))
-  (segment (start 128.905 88.267792) (end 128.905 86.995) (width 0.5) (layer "B.Cu") (net 15))
-  (segment (start 92.71 90.805) (end 126.367792 90.805) (width 0.5) (layer "B.Cu") (net 15))
-  (segment (start 126.367792 90.805) (end 128.905 88.267792) (width 0.5) (layer "B.Cu") (net 15))
-  (segment (start 92.075 91.44) (end 92.71 90.805) (width 0.5) (layer "B.Cu") (net 15))
+  (segment (start 102.235 89.535) (end 100.33 87.63) (width 0.5) (layer "B.Cu") (net 14))
+  (segment (start 93.345 87.63) (end 92.075 88.9) (width 0.5) (layer "B.Cu") (net 14))
+  (segment (start 100.33 87.63) (end 93.345 87.63) (width 0.5) (layer "B.Cu") (net 14))
+  (segment (start 127 91.44) (end 92.075 91.44) (width 0.5) (layer "B.Cu") (net 15))
+  (segment (start 128.905 89.535) (end 127 91.44) (width 0.5) (layer "B.Cu") (net 15))
   (zone (net 1) (net_name "GND") (layers "F&B.Cu") (hatch edge 0.508)
     (connect_pads (clearance 0.508))
